Commit message: mod mass params

File: urdf/simple_bipedal.urdf (robot description, URDF)
Before this commit: robot simple_bipedal, 13 links, 12 joints
Links:
- link ankle_pitch_left_link: mass 13.3431533790223 -> 1.33431533790223
- link ankle_pitch_right_link: mass 13.3431533790223 -> 1.33431533790223
- link ankle_roll_left_link: mass 4.64559018505733 -> 0.464559018505733
- link ankle_roll_right_link: mass 4.64559018505733 -> 0.464559018505733
- link base_link: mass 104.073975462643 -> 10.4073975462643
- link hip_pitch_left_link: mass 8.17782778579702 -> 0.817782778579702
- link hip_pitch_right_link: mass 8.17782778579702 -> 0.817782778579702
- link hip_roll_left_link: mass 6.12916564770063 -> 0.612916564770063
- link hip_roll_right_link: mass 6.12916564770063 -> 0.612916564770063
- link hip_yaw_left_link: mass 15.9288324363201 -> 1.59288324363201
- link hip_yaw_right_link: mass 15.9288324363201 -> 1.59288324363201
- link knee_pitch_left_link: mass 17.3220695885815 -> 1.73220695885815
- link knee_pitch_right_link: mass 17.3220695885815 -> 1.73220695885815

Commit message: joint limits

File: urdf/simple_bipedal.urdf (robot description, URDF)
Before this commit: robot simple_bipedal, 13 links, 12 joints
Joints:
- joint ankle_pitch_left_joint: limit (none) -> lower=-1.57 upper=1.57 effort=100.0 velocity=10.0
- joint ankle_pitch_right_joint: limit (none) -> lower=-1.57 upper=1.57 effort=100.0 velocity=10.0
- joint ankle_roll_left_joint: limit (none) -> lower=-1.57 upper=1.57 effort=100.0 velocity=10.0
- joint ankle_roll_right_joint: limit (none) -> lower=-1.57 upper=1.57 effort=100.0 velocity=10.0
- joint hip_pitch_left_joint: limit (none) -> lower=-1.57 upper=1.57 effort=100.0 velocity=10.0
- joint hip_pitch_right_joint: limit (none) -> lower=-1.57 upper=1.57 effort=100.0 velocity=10.0
- joint hip_roll_left_joint: limit (none) -> lower=-1.57 upper=1.57 effort=100.0 velocity=10.0
- joint hip_roll_right_joint: limit (none) -> lower=-1.57 upper=1.57 effort=100.0 velocity=10.0
- joint hip_yaw_left_joint: limit (none) -> lower=-1.57 upper=1.57 effort=100.0 velocity=10.0
- joint hip_yaw_right_joint: limit (none) -> lower=-1.57 upper=1.57 effort=100.0 velocity=10.0
- joint knee_pitch_left_joint: limit (none) -> lower=-1.57 upper=1.57 effort=100.0 velocity=10.0
- joint knee_pitch_right_joint: limit (none) -> lower=-1.57 upper=1.57 effort=100.0 velocity=10.0

Commit message: modify model

File: urdf/simple_bipedal.urdf (robot description, URDF)
Before this commit: robot simple_bipedal, 13 links, 12 joints
Links:
- link ankle_pitch_left_link: mass 1.33431533790223 -> 1.15921855254247
- link ankle_pitch_right_link: mass 1.33431533790223 -> 1.15921855254247
- link ankle_roll_left_link: mass 0.464559018505733 -> 0.427694789453883
- link ankle_roll_right_link: mass 0.464559018505733 -> 0.42769
- link base_link: mass 10.4073975462643 -> 10.167
- link hip_pitch_left_link: mass 0.817782778579702 -> 0.664887687236356
- link hip_pitch_right_link: mass 0.817782778579702 -> 0.664887687236356
- link hip_roll_left_link: mass 0.612916564770063 -> 0.530800065725118
- link hip_roll_right_link: mass 0.612916564770063 -> 0.530800065725118
- link hip_yaw_left_link: mass 1.59288324363201 -> 1.36383246641991
- link hip_yaw_right_link: mass 1.59288324363201 -> 1.36383246641991
- link knee_pitch_left_link: mass 1.73220695885815 -> 1.50270730941549
- link knee_pitch_right_link: mass 1.73220695885815 -> 1.50270730941549
Joints:
- joint ankle_pitch_left_joint: limit lower=-1.57 upper=1.57 effort=100.0 velocity=10.0 -> lower=-1.57 upper=1.57 effort=100 velocity=10
- joint ankle_pitch_right_joint: limit lower=-1.57 upper=1.57 effort=100.0 velocity=10.0 -> lower=-1.57 upper=1.57 effort=100 velocity=10
- joint ankle_roll_left_joint: limit lower=-1.57 upper=1.57 effort=100.0 velocity=10.0 -> lower=-1.57 upper=1.57 effort=100 velocity=10
- joint ankle_roll_right_joint: limit lower=-1.57 upper=1.57 effort=100.0 velocity=10.0 -> lower=-1.57 upper=1.57 effort=100 velocity=10
- joint hip_pitch_left_joint: limit lower=-1.57 upper=1.57 effort=100.0 velocity=10.0 -> lower=-1.57 upper=1.57 effort=100 velocity=10
- joint hip_pitch_right_joint: limit lower=-1.57 upper=1.57 effort=100.0 velocity=10.0 -> lower=-1.57 upper=1.57 effort=100 velocity=10
- joint hip_roll_left_joint: limit lower=-1.57 upper=1.57 effort=100.0 velocity=10.0 -> lower=-1.57 upper=1.57 effort=100 velocity=10
- joint hip_roll_right_joint: limit lower=-1.57 upper=1.57 effort=100.0 velocity=10.0 -> lower=-1.57 upper=1.57 effort=100 velocity=10
- joint hip_yaw_left_joint: limit lower=-1.57 upper=1.57 effort=100.0 velocity=10.0 -> lower=-1.57 upper=1.57 effort=100 velocity=10
- joint hip_yaw_right_joint: limit lower=-1.57 upper=1.57 effort=100.0 velocity=10.0 -> lower=-1.57 upper=1.57 effort=100 velocity=10
- joint knee_pitch_left_joint: limit lower=-1.57 upper=1.57 effort=100.0 velocity=10.0 -> lower=-1.57 upper=1.57 effort=100 velocity=10
- joint knee_pitch_right_joint: limit lower=-1.57 upper=1.57 effort=100.0 velocity=10.0 -> lower=-1.57 upper=1.57 effort=100 velocity=10
